File: board/board2/board2.sch (KiCad schematic (older format))
At the start: 7 parts, among them J1 11-PIN HDR, J2 MITSU_AC, J3 11-PIN HDR, U1 TXB0104D

Commit message: Commit the old board changes for posterity
Parts:
- removed J1, J3: 11-PIN HDR, Connector_PinSocket_2.54mm:PinSocket_1x11_P2.54mm_Vertical, symbol Connector:Conn_01x11_Female
- added C1, C2, C3: 10uF, Capacitor_SMD:C_0805_2012Metric_Pad1.15x1.40mm_HandSolder, symbol Device:C
- added D1: RED, digikey-footprints:LED_2-SMD_No_Lead_1.7x0.8mm, symbol Device:LED
- added D2, D3: D_Schottky, Diode_SMD:D_SOD-123F, symbol Device:D_Schottky
- added J1: FTDI, Connector_PinHeader_2.54mm:PinHeader_1x06_P2.54mm_Vertical, symbol Connector:Conn_01x06_Male
- added J2: DEBUG, Connector_PinHeader_2.54mm:PinHeader_1x02_P2.54mm_Vertical, symbol Connector:Conn_01x02_Male
- added MOD1: ESP-12S, digikey-footprints:WIFI_Module_ESP8266_2491, symbol dk_RF-Transceiver-Modules:2491
- added R2, R3, R4, R5, R6, R9: 10K, Resistor_SMD:R_0603_1608Metric_Pad1.05x0.95mm_HandSolder, symbol Device:R
- added R7: 1K8, Resistor_SMD:R_0603_1608Metric_Pad1.05x0.95mm_HandSolder, symbol Device:R
- added R8: 3K3, Resistor_SMD:R_0603_1608Metric_Pad1.05x0.95mm_HandSolder, symbol Device:R
- added SW1, SW2, SW3: SW_Push, Button_Switch_SMD:SW_SPST_KMR2, symbol Switch:SW_Push
- added U1: AP2114H-3_3TRG1, digikey-footprints:SOT-223, symbol dk_PMIC-Voltage-Regulators-Linear:AP2114H-3_3TRG1
- R1: value 10K -> 1K
- renumbered C1 to C4, C2 to C5, J2 to J3, U1 to U2
Connections:
- net labels added: CH_PD, GPIO0, GPIO12, GPIO13, GPIO14, GPIO15, GPIO16, GPIO2, RESET, RX0*, RX0*_5V, TX0*, TX0*_5V, TX1, VBUS, VCC, VPP
- net labels removed: +5V, EN, RX0_5V, TX0_5V
- wire segments 40 -> 93
- no-connect marks 19 -> 10
