File: pcb/mitsu-huzzah-interface-board.sch (KiCad schematic (older format))
At the start: 11 parts, among them J1 AIRCON, J2 DEBUG, SW1 KMR2, U1 TXB0102DCUT

Commit message: Update the PCB with a bigger level shifter
Parts:
- removed U1: TXB0102DCUT, Package_SO:VSSOP-8_2.4x2.1mm_P0.5mm, symbol Logic_LevelTranslator:TXB0102DCU
- added U1: TXB0104DR, Package_SO:SOIC-14_3.9x8.7mm_P1.27mm, symbol Logic_LevelTranslator:TXB0104D

Commit message: Update voltage divider resistor values
2K2/3K3 gives a 3V output too, and I didn't want to wait for stock on
the old values.
Parts:
- R1: value 3K9 -> 2K2
- R2: value 6K8 -> 3K3
Changed lines of the file:
@@
 EESchema Schematic File Version 4
+LIBS:mitsu-huzzah-interface-board-cache
 EELAYER 26 0
 EELAYER END
@@
 P 3700 5050
 F 0 "R1" H 3770 5096 50  0000 L CNN
-F 1 "3K9" V 3700 5050 50  0000 C CNN
+F 1 "2K2" V 3700 5050 50  0000 C CNN
 F 2 "Resistor_SMD:R_0603_1608Metric_Pad1.05x0.95mm_HandSolder" V 3630 5050 50  0001 C CNN
 F 3 "~" H 3700 5050 50  0001 C CNN
@@
 P 3700 5750
 F 0 "R2" H 3770 5796 50  0000 L CNN
-F 1 "6K8" V 3700 5750 50  0000 C CNN
+F 1 "3K3" V 3700 5750 50  0000 C CNN
 F 2 "Resistor_SMD:R_0603_1608Metric_Pad1.05x0.95mm_HandSolder" V 3630 5750 50  0001 C CNN
 F 3 "~" H 3700 5750 50  0001 C CNN

Commit message: Change design to a completely custom PCB
No more adafruit HUZZAH, instead build a custom PCB for an ESP-12S module.
Parts:
- removed A1: HUZZAH, mitsu-huzzah-interface-footprints:Adafruit_HUZZAH_ESP8266_breakout_revA_WithMountingHoles, symbol MCU_Module:Adafruit_HUZZAH_ESP8266_breakout
- removed U1: TXB0104DR, Package_SO:SOIC-14_3.9x8.7mm_P1.27mm, symbol Logic_LevelTranslator:TXB0104D
- added C1, C2: 10uF, Capacitor_SMD:C_0603_1608Metric_Pad1.05x0.95mm_HandSolder, symbol Device:C
- added D1, D2: MBR120, Diode_SMD:D_SOD-123F, symbol Device:D_Schottky
- added D3: RED, LED_SMD:LED_0805_2012Metric_Pad1.15x1.40mm_HandSolder, symbol Device:LED
- added D4: MMSD914, Diode_SMD:D_SOD-123, symbol Diode:MMSD914
- added J3: FTDI, Connector_PinHeader_2.54mm:PinHeader_1x06_P2.54mm_Vertical, symbol Connector:Conn_01x06_Male
- added MOD1: 2491, digikey-footprints:WIFI_Module_ESP8266_2491, symbol dk_RF-Transceiver-Modules:2491
- added R10, R2, R3, R8, R9: 10K, Resistor_SMD:R_0603_1608Metric_Pad1.05x0.95mm_HandSolder, symbol Device:R
- added R7: 1K, Resistor_SMD:R_0603_1608Metric_Pad1.05x0.95mm_HandSolder, symbol Device:R
- added SW2, SW3: KMR2, mitsu-huzzah-interface-footprints:SW_SPST_KMR2, symbol Switch:SW_Push
- added U1: AP2112K-3.3TRG1, digikey-footprints:SOT-753, symbol mitsu-huzzah-interface:AP2112K-3.3TRG1
- added U2: TXB0102DCU, Package_SO:VSSOP-8_2.4x2.1mm_P0.5mm, symbol Logic_LevelTranslator:TXB0102DCU
- J1: footprint Connector_JST:JST_PH_S4B-PH-K_1x04_P2.00mm_Horizontal -> agg:S04B-PASK-2
- R1: renamed from R3; value 1K -> 10K
- R4: value 1K -> 10K
- SW1: footprint Button_Switch_SMD:SW_SPST_KMR2 -> mitsu-huzzah-interface-footprints:SW_SPST_KMR2
- renumbered C1 to C3, C2 to C4, R1 to R5, R2 to R6
Connections:
- net labels added: CH_PD, FTDI_5V, FTDI_GND, FTDI_RX, FTDI_TX, GPIO0, GPIO13, GPIO15, GPIO2, RESET, RXD0, RXD0*, RXD0*_5V, TXD0, TXD0*, TXD0*_5V
- net labels removed: RX0*, RX0*_5V, TX0*, TX0*_5V, TX1
- wire segments 43 -> 82
- no-connect marks 10 -> 5
